Commit message: Fix xacro macro args and ParameterValue wrapping for Foxy
- urdf: remove invalid 'name', 'parent', 'robot_ip', script params from
  xacro:ur_robot call -- use actual macro signature from ur_description
- both launch files: wrap Command() in ParameterValue(..., value_type=str)
  to prevent YAML parser choking on colons inside URDF XML strings

System now launches cleanly: robot_state_publisher loads all 14 links
including camera_link, move_group loads robot model successfully.

File: src/simulation/urdf/ur10e_with_realsense.urdf.xacro (robot description, xacro)
@@ -2,13 +2,12 @@
 <robot xmlns:xacro="http://wiki.ros.org/xacro" name="ur10e_realsense">
   <!-- UR10e parameters -->
-  <xacro:arg name="ur_type"           default="ur10e"/>
-  <xacro:arg name="prefix"            default=""/>
-  <xacro:arg name="use_fake_hardware" default="false"/>
+  <xacro:arg name="ur_type"              default="ur10e"/>
+  <xacro:arg name="prefix"               default=""/>
+  <xacro:arg name="use_fake_hardware"    default="false"/>
   <xacro:arg name="fake_sensor_commands" default="false"/>
-  <xacro:arg name="robot_ip"          default="0.0.0.0"/>
-  <xacro:arg name="safety_limits"     default="true"/>
-  <xacro:arg name="safety_pos_margin" default="0.15"/>
-  <xacro:arg name="safety_k_position" default="20"/>
-  <!-- UR description paths -->
+  <xacro:arg name="safety_limits"        default="true"/>
+  <xacro:arg name="safety_pos_margin"    default="0.15"/>
+  <xacro:arg name="safety_k_position"    default="20"/>
+  <!-- UR description parameter files -->
   <xacro:arg name="joint_limit_params"
     default="$(find ur_description)/config/$(arg ur_type)/joint_limits.yaml"/>
@@ -19,24 +18,11 @@
   <xacro:arg name="visual_params"
     default="$(find ur_description)/config/$(arg ur_type)/visual_parameters.yaml"/>
-  <!-- UR robot driver resources (needed even in fake mode) -->
-  <xacro:arg name="script_filename"
-    default="$(find ur_robot_driver)/resources/ros_control.urscript"/>
-  <xacro:arg name="input_recipe_filename"
-    default="$(find ur_robot_driver)/resources/rtde_input_recipe.txt"/>
-  <xacro:arg name="output_recipe_filename"
-    default="$(find ur_robot_driver)/resources/rtde_output_recipe.txt"/>
   <!-- Include UR macro -->
   <xacro:include filename="$(find ur_description)/urdf/ur_macro.xacro"/>
-  <!-- Instantiate UR10e arm, mounted at world origin -->
+  <!-- World link — fixed base for the robot -->
   <link name="world"/>
-  <joint name="world_to_base" type="fixed">
-    <parent link="world"/>
-    <child  link="$(arg prefix)base_link"/>
-    <origin xyz="0 0 0" rpy="0 0 0"/>
-  </joint>
+  <!-- Instantiate UR10e arm -->
   <xacro:ur_robot
-    name="$(arg ur_type)"
-    tf_prefix="$(arg prefix)"
-    parent="world"
+    prefix="$(arg prefix)"
     joint_limits_parameters_file="$(arg joint_limit_params)"
     kinematics_parameters_file="$(arg kinematics_params)"
@@ -47,28 +33,21 @@
     safety_k_position="$(arg safety_k_position)"
     use_fake_hardware="$(arg use_fake_hardware)"
-    fake_sensor_commands="$(arg fake_sensor_commands)"
-    script_filename="$(arg script_filename)"
-    input_recipe_filename="$(arg input_recipe_filename)"
-    output_recipe_filename="$(arg output_recipe_filename)"
-    robot_ip="$(arg robot_ip)">
+    fake_sensor_commands="$(arg fake_sensor_commands)"/>
+  <!-- Fix robot base to world -->
+  <joint name="world_to_base" type="fixed">
+    <parent link="world"/>
+    <child  link="$(arg prefix)base_link"/>
     <origin xyz="0 0 0" rpy="0 0 0"/>
-  </xacro:ur_robot>
+  </joint>
   <!-- ═══════════════════════════════════════════════════════════════
-       RealSense D435 mount — attached to tool0 (end-effector flange)
-       Camera is mounted pointing downward, offset 5 cm in Z
+       RealSense D435 — mounted at tool0 pointing downward
   ════════════════════════════════════════════════════════════════════ -->
   <link name="camera_link">
     <visual>
-      <geometry>
-        <box size="0.025 0.090 0.025"/>
-      </geometry>
-      <material name="dark_grey">
-        <color rgba="0.2 0.2 0.2 1.0"/>
-      </material>
+      <geometry><box size="0.025 0.090 0.025"/></geometry>
+      <material name="dark_grey"><color rgba="0.2 0.2 0.2 1.0"/></material>
     </visual>
     <collision>
-      <geometry>
-        <box size="0.025 0.090 0.025"/>
-      </geometry>
+      <geometry><box size="0.025 0.090 0.025"/></geometry>
     </collision>
     <inertial>
@@ -80,8 +59,8 @@
     <parent link="$(arg prefix)tool0"/>
     <child  link="camera_link"/>
-    <!-- 5cm down from flange, rotated so camera Z points forward (away from robot) -->
+    <!-- 5 cm below flange, rotated so camera Z points forward -->
     <origin xyz="0 0 0.05" rpy="0 1.5708 0"/>
   </joint>
-  <!-- Optical frame: ROS convention — Z forward, X right, Y down -->
+  <!-- Optical frame: Z forward, X right, Y down (ROS convention) -->
   <link name="camera_color_optical_frame"/>
   <joint name="camera_color_optical_joint" type="fixed">
@@ -90,5 +69,5 @@
     <origin xyz="0 0 0" rpy="-1.5708 0 -1.5708"/>
   </joint>
-  <!-- Gazebo camera sensor plugin (RGB + Depth) -->
+  <!-- Gazebo depth camera plugin — publishes on /camera/* matching real driver -->
   <gazebo reference="camera_link">
     <sensor type="depth" name="realsense_d435">
@@ -96,5 +75,5 @@
       <update_rate>30.0</update_rate>
       <camera name="realsense">
-        <horizontal_fov>1.2217</horizontal_fov>  <!-- ~70 deg, D435 spec -->
+        <horizontal_fov>1.2217</horizontal_fov>
         <image>
           <width>640</width>
@@ -102,15 +81,7 @@
           <format>R8G8B8</format>
         </image>
-        <clip>
-          <near>0.1</near>
-          <far>10.0</far>
-        </clip>
-        <noise>
-          <type>gaussian</type>
-          <mean>0.0</mean>
-          <stddev>0.001</stddev>
-        </noise>
+        <clip><near>0.1</near><far>10.0</far></clip>
+        <noise><type>gaussian</type><mean>0.0</mean><stddev>0.001</stddev></noise>
       </camera>
-      <!-- Publishes on same topics as the real RealSense driver -->
       <plugin name="realsense_plugin" filename="libgazebo_ros_camera.so">
         <ros>
@@ -123,5 +94,4 @@
         <camera_name>realsense_d435</camera_name>
         <frame_name>camera_color_optical_frame</frame_name>
-        <hack_baseline>0.0</hack_baseline>
         <min_depth>0.1</min_depth>
         <max_depth>10.0</max_depth>

Commit message: Add Robotiq 2F-85 gripper + RealSense wrist bracket mount
- Add ros2_robotiq_gripper as git submodule (PickNikRobotics/ros2_robotiq_gripper)
- URDF: tool0 -> ur_to_robotiq adapter -> Robotiq 2F-85 gripper
- URDF: tool0 -> camera_bracket_link (side wrist bracket) -> RealSense D435
  Camera offset 8cm to side, 3cm back, pitched 30deg down toward workspace
  Camera no longer blocks gripper TCP

File: src/simulation/urdf/ur10e_with_realsense.urdf.xacro (robot description, xacro)
@@ -1,5 +1,13 @@
 <?xml version="1.0"?>
 <robot xmlns:xacro="http://wiki.ros.org/xacro" name="ur10e_realsense">
-  <!-- UR10e parameters -->
+  <!-- ════════════════════════════════════════════════════════════════
+       UR10e + Robotiq 2F-85 gripper + RealSense D435 (wrist-mounted)
+       Mount layout (all attached to tool0):
+         tool0 ──► ur_to_robotiq adapter ──► Robotiq 2F-85 (TCP at ~170mm below tool0)
+         tool0 ──► camera_bracket_link   ──► camera_link
+                   (offset: 0.03m back along arm, 0.08m away from gripper axis)
+                   (pitched 30° down to see workspace under gripper)
+  ═══════════════════════════════════════════════════════════════════ -->
+  <!-- ── UR10e parameters ─────────────────────────────────────────── -->
   <xacro:arg name="ur_type"              default="ur10e"/>
   <xacro:arg name="prefix"               default=""/>
@@ -9,5 +17,4 @@
   <xacro:arg name="safety_pos_margin"    default="0.15"/>
   <xacro:arg name="safety_k_position"    default="20"/>
-  <!-- UR description parameter files -->
   <xacro:arg name="joint_limit_params"
     default="$(find ur_description)/config/$(arg ur_type)/joint_limits.yaml"/>
@@ -18,9 +25,11 @@
   <xacro:arg name="visual_params"
     default="$(find ur_description)/config/$(arg ur_type)/visual_parameters.yaml"/>
-  <!-- Include UR macro -->
+  <!-- ── Includes ─────────────────────────────────────────────────── -->
   <xacro:include filename="$(find ur_description)/urdf/ur_macro.xacro"/>
-  <!-- World link — fixed base for the robot -->
+  <xacro:include filename="$(find robotiq_description)/urdf/ur_to_robotiq_adapter.urdf.xacro"/>
+  <xacro:include filename="$(find robotiq_description)/urdf/robotiq_2f_85_macro.urdf.xacro"/>
+  <!-- ── World link ───────────────────────────────────────────────── -->
   <link name="world"/>
-  <!-- Instantiate UR10e arm -->
+  <!-- ── UR10e arm ────────────────────────────────────────────────── -->
   <xacro:ur_robot
     prefix="$(arg prefix)"
@@ -34,5 +43,4 @@
     use_fake_hardware="$(arg use_fake_hardware)"
     fake_sensor_commands="$(arg fake_sensor_commands)"/>
-  <!-- Fix robot base to world -->
   <joint name="world_to_base" type="fixed">
     <parent link="world"/>
@@ -40,14 +48,61 @@
     <origin xyz="0 0 0" rpy="0 0 0"/>
   </joint>
-  <!-- ═══════════════════════════════════════════════════════════════
-       RealSense D435 — mounted at tool0 pointing downward
-  ════════════════════════════════════════════════════════════════════ -->
+  <!-- ── UR-to-Robotiq adapter plate (at tool0 flange) ───────────── -->
+  <xacro:ur_to_robotiq
+    prefix="$(arg prefix)"
+    parent="$(arg prefix)tool0"
+    child="$(arg prefix)robotiq_85_base_link"/>
+  <!-- ── Robotiq 2F-85 gripper ────────────────────────────────────── -->
+  <xacro:robotiq_gripper
+    name="RobotiqHandE"
+    prefix="$(arg prefix)"
+    parent="$(arg prefix)robotiq_85_base_link"
+    use_fake_hardware="$(arg use_fake_hardware)"
+    sim_gazebo="true">
+    <origin xyz="0 0 0" rpy="0 0 0"/>
+  </xacro:robotiq_gripper>
+  <!-- ── Camera bracket (rigid, attached to tool0) ─────────────────
+       Bracket sits 3cm back along the Z axis of tool0 (toward the arm)
+       and 8cm offset along Y (to the side of the gripper axis).
+       This clears the gripper body and gives a clear view of the workspace.
+  ──────────────────────────────────────────────────────────────────── -->
+  <link name="camera_bracket_link">
+    <visual>
+      <geometry><box size="0.02 0.02 0.10"/></geometry>
+      <material name="bracket_grey"><color rgba="0.5 0.5 0.5 1.0"/></material>
+    </visual>
+    <inertial>
+      <mass value="0.05"/>
+      <inertia ixx="1e-5" ixy="0" ixz="0" iyy="1e-5" iyz="0" izz="1e-5"/>
+    </inertial>
+  </link>
+  <gazebo reference="camera_bracket_link">
+    <material>Gazebo/Grey</material>
+  </gazebo>
+  <joint name="camera_bracket_joint" type="fixed">
+    <parent link="$(arg prefix)tool0"/>
+    <child  link="camera_bracket_link"/>
+    <!--
+      xyz: 0.08m offset in Y (side of gripper), -0.03m back in Z (toward arm body)
+      rpy: rotate 30 degrees around X so camera looks down toward workspace
+    -->
+    <origin xyz="0 0.08 -0.03" rpy="-0.5236 0 0"/>
+  </joint>
+  <!-- ── RealSense D435 body ──────────────────────────────────────── -->
   <link name="camera_link">
+    <!-- Main body: 90mm × 25mm × 25mm -->
     <visual>
-      <geometry><box size="0.025 0.090 0.025"/></geometry>
-      <material name="dark_grey"><color rgba="0.2 0.2 0.2 1.0"/></material>
+      <origin xyz="0 0 0" rpy="0 0 0"/>
+      <geometry><box size="0.090 0.025 0.025"/></geometry>
+      <material name="realsense_body"><color rgba="0.1 0.1 0.1 1.0"/></material>
+    </visual>
+    <!-- Blue lens strip on front face -->
+    <visual>
+      <origin xyz="0.020 0.0 0.014" rpy="0 0 0"/>
+      <geometry><box size="0.060 0.025 0.003"/></geometry>
+      <material name="lens_blue"><color rgba="0.2 0.5 0.9 1.0"/></material>
     </visual>
     <collision>
-      <geometry><box size="0.025 0.090 0.025"/></geometry>
+      <geometry><box size="0.090 0.025 0.025"/></geometry>
     </collision>
     <inertial>
@@ -56,11 +111,14 @@
     </inertial>
   </link>
-  <joint name="camera_mount_joint" type="fixed">
-    <parent link="$(arg prefix)tool0"/>
+  <gazebo reference="camera_link">
+    <material>Gazebo/DarkGrey</material>
+  </gazebo>
+  <joint name="camera_link_joint" type="fixed">
+    <parent link="camera_bracket_link"/>
     <child  link="camera_link"/>
-    <!-- 5 cm below flange, rotated so camera Z points forward -->
-    <origin xyz="0 0 0.05" rpy="0 1.5708 0"/>
+    <!-- Camera sits at the end of the bracket, lens facing workspace -->
+    <origin xyz="0 0 -0.05" rpy="0 0 0"/>
   </joint>
-  <!-- Optical frame: Z forward, X right, Y down (ROS convention) -->
+  <!-- Optical frame: Z forward, X right, Y down (ROS camera convention) -->
   <link name="camera_color_optical_frame"/>
   <joint name="camera_color_optical_joint" type="fixed">
@@ -69,5 +127,5 @@
     <origin xyz="0 0 0" rpy="-1.5708 0 -1.5708"/>
   </joint>
-  <!-- Gazebo depth camera plugin — publishes on /camera/* matching real driver -->
+  <!-- ── Gazebo depth camera sensor ───────────────────────────────── -->
   <gazebo reference="camera_link">
     <sensor type="depth" name="realsense_d435">
@@ -81,10 +139,9 @@
           <format>R8G8B8</format>
         </image>
-        <clip><near>0.1</near><far>10.0</far></clip>
+        <clip><near>0.1</near><far>3.0</far></clip>
         <noise><type>gaussian</type><mean>0.0</mean><stddev>0.001</stddev></noise>
       </camera>
       <plugin name="realsense_plugin" filename="libgazebo_ros_camera.so">
         <ros>
-          <!-- Publish directly on /camera/color/* and /camera/aligned_depth_to_color/* -->
           <namespace>/camera</namespace>
           <remapping>realsense_d435/image_raw:=color/image_raw</remapping>
@@ -96,5 +153,5 @@
         <frame_name>camera_color_optical_frame</frame_name>
         <min_depth>0.1</min_depth>
-        <max_depth>10.0</max_depth>
+        <max_depth>3.0</max_depth>
       </plugin>
     </sensor>

Commit message: Fix ros2_control compatibility for Foxy simulation
OpaqueFunction in sim_gazebo.launch.py post-processes the URDF:
- Strip <gpio> blocks (added in newer ros2_control, not in Foxy)
- Replace mock_components/GenericSystem with fake_components/GenericSystem
  (Robotiq macro uses newer naming; Foxy only has fake_components)

Rebuild workspace without booksros2_ws in chain (install/setup.bash
now only chains to /opt/ros/foxy, not booksros2_ws).

Robotiq gripper: sim_gazebo=false (was triggering ign_ros2_control/
IgnitionSystem for Gazebo Ignition, not Gazebo Classic)

Result: all 9 nodes up, controllers active at 500Hz, camera publishing.

File: src/simulation/urdf/ur10e_with_realsense.urdf.xacro (robot description, xacro)
@@ -59,6 +59,6 @@
     prefix="$(arg prefix)"
     parent="$(arg prefix)robotiq_coupler_link"
-    use_fake_hardware="$(arg use_fake_hardware)"
-    sim_gazebo="true">
+    use_fake_hardware="true"
+    sim_gazebo="false">
     <origin xyz="0 0 0" rpy="0 0 0"/>
   </xacro:robotiq_gripper>
@@ -73,4 +73,7 @@
       <material name="bracket_grey"><color rgba="0.5 0.5 0.5 1.0"/></material>
     </visual>
+    <collision>
+      <geometry><box size="0.02 0.02 0.10"/></geometry>
+    </collision>
     <inertial>
       <mass value="0.05"/>

Commit message: Switch to headless gzserver — eliminates gzclient crash cascade
gzclient was crashing with boost::shared_ptr assertion in depth camera
rendering code, which caused the launch system to SIGTERM gzserver.
Running gzserver-only (no GUI window) keeps gzserver stable and camera
topics publishing continuously. RViz is used for visualization instead.

File: src/simulation/urdf/ur10e_with_realsense.urdf.xacro (robot description, xacro)
@@ -88,8 +88,10 @@
     <child  link="camera_bracket_link"/>
     <!--
-      xyz: 0.08m offset in Y (side of gripper), -0.03m back in Z (toward arm body)
-      rpy: rotate 30 degrees around X so camera looks down toward workspace
+      Camera mounted behind the flange, offset to the side for gripper clearance.
+      xyz: -0.06m back in Z (toward arm body), +0.05m to the side (Y)
+      rpy: +30° pitch so camera looks FORWARD along the gripper approach axis
+           (same direction as gripper — toward the object being picked)
     -->
-    <origin xyz="0 0.08 -0.03" rpy="-0.5236 0 0"/>
+    <origin xyz="0 0.05 -0.06" rpy="0.5236 0 0"/>
   </joint>
   <!-- ── RealSense D435 body ──────────────────────────────────────── -->
